File: PCB/Battle_bot_pcb.kicad_pcb (KiCad board)
At the start: 4 copper layers, 45.8 x 30.4 mm, 64 parts, among them J1 USB_C_Receptacle_USB2.0, J2 Conn_01x04, J3 Conn_01x02, J4 Conn_01x02, J5 Conn_01x02, J6 Conn_01x02, J7 Conn_01x02, Q1 AO3401A, SW1 Reset, SW2 Boot, U1 LSM6DS3, U2 ESP32-S3, U3 USBLC6-2P6, U4 LTC4412xS6, U5 DRV8833RTY, U6 TPS62172DSG, Y1 40MHz

Commit message: I/O header
Parts:
- added J8: Conn_01x04, Connector_PinHeader_2.54mm:PinHeader_1x04_P2.54mm_Vertical, F.Cu at (145.1, 85.0)
- moved D2 25.1 mm to (158.9, 108.5), turned to 0 degrees
- moved R2 23.1 mm to (155.8, 109.0)
- moved R5 0.73 mm to (155.8, 87.2)
- moved C1 0.38 mm to (134.7, 85.2)
- moved D1 0.15 mm to (137.6, 84.7)
Connections:
- U2 pad 38: unconnected-(U2-GPIO33-Pad38) -> Net-(J8-Pin_4)
- U2 pad 39: unconnected-(U2-GPIO34-Pad39) -> Net-(J8-Pin_3)
- U2 pad 40: unconnected-(U2-GPIO35-Pad40) -> Net-(J8-Pin_2)
- U2 pad 41: unconnected-(U2-GPIO36-Pad41) -> /DEBUG
- U2 pad 42: unconnected-(U2-GPIO37-Pad42) -> Net-(J8-Pin_1)
Routing:
- net Net-(J8-Pin_3): track 0.00 -> 16.3 mm, vias 0 -> 1
- net Net-(J8-Pin_4): track 0.00 -> 16.1 mm, vias 0 -> 1
- net Net-(J8-Pin_2): track 0.00 -> 14.4 mm, vias 0 -> 1
- net Net-(J8-Pin_1): track 0.00 -> 14.0 mm, vias 0 -> 1
- net +3.3V: track 16.6 -> 18.3 mm, vias 11 -> 12
- net +BATT: track 37.2 -> 36.5 mm
- net GND: track 33.6 -> 33.5 mm, vias 86 -> 85
Other:
- board text added: "I/O"

Commit message: small changes
Parts:
- removed the C15 at (147.8, 90.4)
- moved R7 0.55 mm to (132.9, 89.6)
- moved R11 0.38 mm to (149.6, 105.4)
- moved D1 0.30 mm to (137.6, 84.4)
- moved C6 0.18 mm to (149.4, 92.8)
- moved C8 0.18 mm to (149.4, 95.0)
- moved C24 0.09 mm to (148.8, 101.8)
- moved L4 0.09 mm to (148.8, 104.0)
Routing:
- net Net-(J8-Pin_4): track 16.1 -> 18.5 mm
- net +5V: track 8.73 -> 9.24 mm
- net GND: track 33.5 -> 33.8 mm, vias 85 -> 82
