File: PCB/Battle_bot_pcb.kicad_pcb (KiCad board)
At the start: 4 copper layers, 45.8 x 30.4 mm, 66 parts, among them J1 UJ2-MIBH2-4-SMT-TR, J10 Conn_01x02, J2 Conn_01x04, J3 Conn_01x02, J4 Conn_01x02, J5 Conn_01x02, J6 Conn_01x02, Q1 AO3401A, SW3 Reset, SW4 Boot, U1 LSM6DS3, U2 LTC4412xS6, U3 USBLC6-2P6, U4 TPS62172DSG, U5 DRV8833RTY, U7 ESP32-S3, Y2 40MHz

Commit message: Production files
Parts:
- J1: value UJ2-MIBH2-4-SMT-TR -> USB_B_Micro; footprint UJ2-MIBH2-4-SMT-TR:CUI_UJ2-MIBH2-4-SMT-TR -> Connector_USB:USB_Micro-B_Molex-105017-0001
- moved J1 0.80 mm to (166.8, 105.3)
Routing:
- net GND: track 42.5 -> 43.8 mm
- net VBUS: track 9.81 -> 9.20 mm
Other:
- board text added: "+"
