File: PCB/io.kicad_sch (KiCad schematic)
At the start: 7 parts, among them J2 Conn_01x04, J3 Conn_01x02, J4 Conn_01x02, U5 DRV8833RTY

Commit message: Production files
Changed lines of the file:
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@@
 	(text "min 16v cap rating"
 		(exclude_from_sim no)
-		(at 107.188 82.804 0)
+		(at 106.934 84.074 0)
 		(effects
 			(font

Commit message: Updates to README
Other:
- note added: "Motor Driver"
Changed lines of the file:
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@@
+		)
+	)
+	(text "Motor Driver"
+		(exclude_from_sim no)
+		(at 194.818 174.498 0)
+		(effects
+			(font
+				(face "KiCad Font")
+				(size 3 3)
+				(thickness 0.6)
+				(bold yes)
+			)
 		)
 	)
@@
 	(label "IN2"
 		(at 142.24 107.95 0)
-		(fields_autoplaced yes)
 		(effects
 			(font
@@
 	(label "IN4"
 		(at 142.24 113.03 0)
-		(fields_autoplaced yes)
 		(effects
 			(font
@@
 	(label "IN[1..4]"
 		(at 128.27 127 180)
-		(fields_autoplaced yes)
 		(effects
 			(font
@@
 	(label "AOUT2"
 		(at 177.8 107.95 0)
-		(fields_autoplaced yes)
 		(effects
 			(font
@@
 	(label "BOUT2"
 		(at 177.8 113.03 0)
-		(fields_autoplaced yes)
 		(effects
 			(font
@@
 	(label "AOUT1"
 		(at 177.8 105.41 0)
-		(fields_autoplaced yes)
 		(effects
 			(font
@@
 	(label "IN1"
 		(at 142.24 105.41 0)
-		(fields_autoplaced yes)
 		(effects
 			(font
@@
 	(label "IN3"
 		(at 142.24 110.49 0)
-		(fields_autoplaced yes)
 		(effects
 			(font
@@
 	(label "BOUT1"
 		(at 177.8 110.49 0)
-		(fields_autoplaced yes)
 		(effects
 			(font
@@
 		(shape output)
 		(at 194.31 96.52 0)
-		(fields_autoplaced yes)
 		(effects
 			(font
@@
 		(shape input)
 		(at 139.7 92.71 180)
-		(fields_autoplaced yes)
 		(effects
 			(font
@@
 		(shape input)
 		(at 121.92 127 180)
-		(fields_autoplaced yes)
 		(effects
 			(font
