File: PCB/_autosave-inverter.kicad_sch (KiCad schematic)
At the start: 36 parts, among them J4 Conn_01x03, Q10 BSC026N08NS5, Q11 BSC026N08NS5, Q12 BSC026N08NS5, Q13 BSC026N08NS5, Q8 BSC026N08NS5, Q9 BSC026N08NS5, U10 ACS711xEXLT-31AB, U11 ACS711xEXLT-31AB, U13 IR2103, U14 ACS725xLCTR-50AB, U15 INA849D, U8 IR2103, U9 IR2103

Commit message: Latest PCB version
Connections:
- net at R37.2, R41.1: now also U15.4 (+); no longer U15.1 (-)
- net at R42.2, R43.1: now also U15.1 (-); no longer U15.3 (Rg)
Other:
- moved on the sheet: R37, R41, R42, R43, U15
Changed lines of the file:
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@@
 	)
 	(junction
-		(at 124.46 163.83)
+		(at 123.19 160.02)
 		(diameter 0)
 		(color 0 0 0 0)
@@
 	)
 	(junction
-		(at 124.46 140.97)
+		(at 123.19 137.16)
 		(diameter 0)
 		(color 0 0 0 0)
@@
 	)
 	(junction
-		(at 124.46 152.4)
+		(at 123.19 148.59)
 		(diameter 0)
 		(color 0 0 0 0)
@@
 	(wire
 		(pts
-			(xy 124.46 139.7) (xy 124.46 140.97)
+			(xy 123.19 135.89) (xy 123.19 137.16)
 		)
 		(stroke
@@
 	(wire
 		(pts
-			(xy 115.57 132.08) (xy 124.46 132.08)
+			(xy 114.3 128.27) (xy 123.19 128.27)
 		)
 		(stroke
@@
 	(wire
 		(pts
-			(xy 114.3 152.4) (xy 124.46 152.4)
+			(xy 113.03 148.59) (xy 123.19 148.59)
 		)
 		(stroke
@@
 	(wire
 		(pts
-			(xy 140.97 140.97) (xy 124.46 140.97)
+			(xy 123.19 137.16) (xy 149.86 137.16)
 		)
 		(stroke
@@
 	(wire
 		(pts
-			(xy 124.46 173.99) (xy 124.46 172.72)
+			(xy 123.19 170.18) (xy 123.19 168.91)
 		)
 		(stroke
@@
 	(wire
 		(pts
-			(xy 124.46 152.4) (xy 124.46 154.94)
+			(xy 123.19 148.59) (xy 123.19 151.13)
 		)
 		(stroke
@@
 	(wire
 		(pts
-			(xy 140.97 148.59) (xy 140.97 140.97)
-		)
-		(stroke
-			(width 0)
-			(type default)
-		)
-	)
-	(wire
-		(pts
 			(xy 81.28 100.33) (xy 81.28 86.36)
 		)
@@
 	(wire
 		(pts
-			(xy 114.3 173.99) (xy 124.46 173.99)
+			(xy 113.03 170.18) (xy 123.19 170.18)
 		)
 		(stroke
@@
 	(wire
 		(pts
-			(xy 124.46 140.97) (xy 124.46 142.24)
+			(xy 123.19 137.16) (xy 123.19 138.43)
 		)
 		(stroke
@@
 	(wire
 		(pts
-			(xy 124.46 163.83) (xy 124.46 165.1)
+			(xy 123.19 160.02) (xy 123.19 161.29)
 		)
 		(stroke
@@
 	(wire
 		(pts
-			(xy 144.78 156.21) (xy 140.97 156.21)
-		)
-		(stroke
-			(width 0)
-			(type default)
-		)
-	)
-	(wire
-		(pts
 			(xy 68.58 143.51) (xy 71.12 143.51)
 		)
@@
 	(wire
 		(pts
-			(xy 140.97 163.83) (xy 124.46 163.83)
+			(xy 139.7 160.02) (xy 123.19 160.02)
 		)
 		(stroke
@@
 	(wire
 		(pts
-			(xy 140.97 156.21) (xy 140.97 163.83)
+			(xy 139.7 147.32) (xy 139.7 160.02)
 		)
 		(stroke
@@
 	(wire
 		(pts
-			(xy 124.46 149.86) (xy 124.46 152.4)
+			(xy 123.19 146.05) (xy 123.19 148.59)
 		)
 		(stroke
@@
 	(wire
 		(pts
-			(xy 144.78 148.59) (xy 140.97 148.59)
-		)
-		(stroke
-			(width 0)
-			(type default)
-		)
-	)
-	(wire
-		(pts
 			(xy 50.8 86.36) (xy 68.58 86.36)
 		)
@@
 	(wire
 		(pts
-			(xy 124.46 162.56) (xy 124.46 163.83)
+			(xy 123.19 158.75) (xy 123.19 160.02)
 		)
 		(stroke
@@
 	(wire
 		(pts
+			(xy 149.86 147.32) (xy 139.7 147.32)
+		)
+		(stroke
+			(width 0)
+			(type default)
+		)
+	)
+	(wire
+		(pts
 			(xy 71.12 69.85) (xy 71.12 63.5)
 		)
@@
 	)
 	(label "B"
-		(at 114.3 152.4 0)
+		(at 113.03 148.59 0)
 		(effects
 			(font
@@
 	)
 	(label "A"
-		(at 115.57 132.08 0)
+		(at 114.3 128.27 0)
 		(effects
 			(font
@@
 	)
 	(label "C"
-		(at 114.3 173.99 0)
+		(at 113.03 170.18 0)
 		(effects
 			(font
@@
 	(symbol
 		(lib_id "Amplifier_Instrumentation:INA849D")
-		(at 152.4 153.67 0)
+		(at 157.48 142.24 0)
+		(mirror x)
 		(unit 1)
 		(exclude_from_sim no)
@@
 		(on_board yes)
 		(dnp no)
-		(fields_autoplaced yes)
 		(property "Reference" "U15"
-			(at 167.64 147.2498 0)
+			(at 172.72 148.6602 0)
 			(effects
 				(font
@@
 		)
 		(property "Value" "INA849D"
-			(at 167.64 149.7898 0)
+			(at 172.72 146.1202 0)
 			(effects
 				(font
@@
 		)
 		(property "Footprint" "Package_SO:SOIC-8_3.9x4.9mm_P1.27mm"
-			(at 152.654 181.102 0)
+			(at 157.734 114.808 0)
 			(effects
 				(font
@@
 		)
 		(property "Datasheet" "https://www.ti.com/lit/ds/symlink/ina849.pdf"
-			(at 152.908 183.642 0)
+			(at 157.988 112.268 0)
 			(effects
 				(font
@@
 		)
 		(property "Description" "Ultra-Low-Noise (1 nV/√Hz), 28 MHz Bandwidth, Instrumentation Amplifier, Supply Range 8V to 36V, SOIC-8"
-			(at 152.4 178.562 0)
+			(at 157.48 117.348 0)
 			(effects
 				(font
@@
 	(symbol
 		(lib_id "Device:R")
-		(at 124.46 168.91 0)
+		(at 123.19 165.1 0)
 		(unit 1)
 		(exclude_from_sim no)
@@
 		(fields_autoplaced yes)
 		(property "Reference" "R43"
-			(at 127 167.6399 0)
+			(at 125.73 163.8299 0)
 			(effects
 				(font
@@
 		)
 		(property "Value" "R"
-			(at 127 170.1799 0)
+			(at 125.73 166.3699 0)
 			(effects
 				(font
@@
 		)
 		(property "Footprint" ""
-			(at 122.682 168.91 90)
+			(at 121.412 165.1 90)
 			(effects
 				(font
@@
 		)
 		(property "Datasheet" "~"
-			(at 124.46 168.91 0)
+			(at 123.19 165.1 0)
 			(effects
 				(font
@@
 		)
 		(property "Description" "Resistor"
-			(at 124.46 168.91 0)
+			(at 123.19 165.1 0)
 			(effects
 				(font
@@
 	(symbol
 		(lib_id "Device:R")
-		(at 124.46 135.89 0)
+		(at 123.19 132.08 0)
 		(unit 1)
 		(exclude_from_sim no)
@@
 		(fields_autoplaced yes)
 		(property "Reference" "R37"
-			(at 127 134.6199 0)
+			(at 125.73 130.8099 0)
 			(effects
 				(font
@@
 		)
 		(property "Value" "R"
-			(at 127 137.1599 0)
+			(at 125.73 133.3499 0)
 			(effects
 				(font
@@
 		)
 		(property "Footprint" ""
-			(at 122.682 135.89 90)
+			(at 121.412 132.08 90)
 			(effects
 				(font
@@
 		)
 		(property "Datasheet" "~"
-			(at 124.46 135.89 0)
+			(at 123.19 132.08 0)
 			(effects
 				(font
@@
 		)
 		(property "Description" "Resistor"
-			(at 124.46 135.89 0)
+			(at 123.19 132.08 0)
 			(effects
 				(font
@@
 	(symbol
 		(lib_id "Device:R")
-		(at 124.46 146.05 0)
+		(at 123.19 142.24 0)
 		(unit 1)
 		(exclude_from_sim no)
@@
 		(fields_autoplaced yes)
 		(property "Reference" "R41"
-			(at 127 144.7799 0)
+			(at 125.73 140.9699 0)
 			(effects
 				(font
@@
 		)
 		(property "Value" "R"
-			(at 127 147.3199 0)
+			(at 125.73 143.5099 0)
 			(effects
 				(font
@@
 		)
 		(property "Footprint" ""
-			(at 122.682 146.05 90)
+			(at 121.412 142.24 90)
 			(effects
 				(font
@@
 		)
 		(property "Datasheet" "~"
-			(at 124.46 146.05 0)
+			(at 123.19 142.24 0)
 			(effects
 				(font
@@
 		)
 		(property "Description" "Resistor"
-			(at 124.46 146.05 0)
+			(at 123.19 142.24 0)
 			(effects
 				(font
@@
 	(symbol
 		(lib_id "Device:R")
-		(at 124.46 158.75 0)
+		(at 123.19 154.94 0)
 		(unit 1)
 		(exclude_from_sim no)
@@
 		(fields_autoplaced yes)
 		(property "Reference" "R42"
-			(at 127 157.4799 0)
+			(at 125.73 153.6699 0)
 			(effects
 				(font
@@
 		)
 		(property "Value" "R"
-			(at 127 160.0199 0)
+			(at 125.73 156.2099 0)
 			(effects
 				(font
@@
 		)
 		(property "Footprint" ""
-			(at 122.682 158.75 90)
+			(at 121.412 154.94 90)
 			(effects
 				(font
@@
 		)
 		(property "Datasheet" "~"
-			(at 124.46 158.75 0)
+			(at 123.19 154.94 0)
 			(effects
 				(font
@@
 		)
 		(property "Description" "Resistor"
-			(at 124.46 158.75 0)
+			(at 123.19 154.94 0)
 			(effects
 				(font
